File: minimouse.kicad_pcb (KiCad board)
At the start: 2 copper layers, 90 x 85 mm, 23 parts, among them J1 Conn_ARM_JTAG_SWD_10, J5 Conn_01x02, M1 N20_encoder, M2 N20_encoder, U1 STM32F030C8Tx, U3 HC-SR04, U4 LP5907MFX-1.2

Commit message: deuxieme commit
Parts:
- added C10: 2.2 uF, Capacitor_SMD:C_0603_1608Metric, F.Cu at (134.0, 67.0)
- added C11: 2.2uF, Capacitor_SMD:C_0603_1608Metric, F.Cu at (155.1, 69.5)
- added C12: 2.2uF, Capacitor_SMD:C_0603_1608Metric, F.Cu at (142.4, 69.5)
- added C7: 2.2 uF, Capacitor_SMD:C_0603_1608Metric, F.Cu at (132.2, 87.4)
- added C8: 2.2 uF, Capacitor_SMD:C_0603_1608Metric, F.Cu at (181.3, 82.2)
- added C9: 2.2 uF, Capacitor_SMD:C_0603_1608Metric, F.Cu at (184.8, 94.9)
- added Cen1: 10 nF, Capacitor_SMD:C_0603_1608Metric, F.Cu at (181.3, 72.1)
- added Crcoff1: 22 nF, Capacitor_SMD:C_0603_1608Metric, F.Cu at (174.6, 67.0)
- added D1: LED, LED_SMD:LED_0603_1608Metric, F.Cu at (154.3, 64.4)
- added J2: Conn_01x06, Connector_PinHeader_2.54mm:PinHeader_1x06_P2.54mm_Vertical, F.Cu at (122.1, 100.0)
- added J3: Conn_01x06, Connector_PinHeader_2.54mm:PinHeader_1x06_P2.54mm_Vertical, F.Cu at (162.7, 100.0)
- added J4: Conn_01x04, Connector_PinHeader_2.54mm:PinHeader_1x04_P2.54mm_Vertical, F.Cu at (127.1, 67.0)
- added R10: 10k, Resistor_SMD:R_0603_1608Metric, F.Cu at (174.6, 77.1)
- added R11: 100, Resistor_SMD:R_0603_1608Metric, F.Cu at (120.3, 72.1)
- added R12: 100, Resistor_SMD:R_0603_1608Metric, F.Cu at (181.3, 84.8)
- added R13: 330, Resistor_SMD:R_0603_1608Metric, F.Cu at (155.1, 67.0)
- added R14: 10k, Resistor_SMD:R_0603_1608Metric, F.Cu at (174.6, 74.6)
- added R15: 100, Resistor_SMD:R_0603_1608Metric, F.Cu at (132.2, 89.9)
- added R16: 100, Resistor_SMD:R_0603_1608Metric, F.Cu at (172.0, 94.9)
- added R17: 100, Resistor_SMD:R_0603_1608Metric, F.Cu at (132.2, 92.4)
- added R18: 100, Resistor_SMD:R_0603_1608Metric, F.Cu at (166.1, 97.5)
- added Ren1: 10k, Resistor_SMD:R_0603_1608Metric, F.Cu at (181.3, 74.6)
- added Roff1: 47 k, Resistor_SMD:R_0603_1608Metric, F.Cu at (174.6, 72.1)
- added Rrcoff1: 1 k, Resistor_SMD:R_0603_1608Metric, F.Cu at (174.6, 69.5)
- added Rsnsa1: 330 m, Resistor_SMD:R_0603_1608Metric, F.Cu at (181.3, 77.1)
- added Rsnsb1: 330 m, Resistor_SMD:R_0603_1608Metric, F.Cu at (181.3, 79.7)
- added U5: STSPIN240, Package_DFN_QFN:VQFN-16-1EP_3x3mm_P0.5mm_EP1.8x1.8mm, F.Cu at (167.5, 78.2)
- moved J1 6.29 mm to (157.6, 83.5)

Commit message: save
Parts:
- moved Rsnsb1 42.4 mm to (144.3, 100.4), turned to -90 degrees
- moved Rsnsa1 37.4 mm to (152.2, 100.6)
- moved Crcoff1 36.5 mm to (155.2, 97.8), turned to 90 degrees
- moved Rrcoff1 36.2 mm to (152.1, 97.8), turned to 90 degrees
- moved Cen1 35.8 mm to (153.6, 94.8), turned to -90 degrees
- moved Ren1 35.5 mm to (152.1, 94.8), turned to -90 degrees
- moved Roff1 33.2 mm to (153.6, 97.8), turned to 90 degrees
- moved R12 32.9 mm to (149.2, 77.5), turned to 90 degrees
- moved U5 28.8 mm to (147.9, 99.3)
- moved C8 28.3 mm to (155.9, 69.7)
- moved R14 28.0 mm to (155.1, 94.8), turned to 90 degrees
- moved R10 25.2 mm to (156.7, 94.8), turned to 90 degrees
- moved C4 19.1 mm to (140.5, 83.9), turned to 180 degrees
- moved C5 17.8 mm to (140.5, 82.4)
- moved C9 14.7 mm to (172.2, 102.6), turned to 180 degrees
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Routing:
- net /mcu/TIM2_CH1: track 0.00 -> 126.9 mm
- net /mcu/TIM2_CH2: track 0.00 -> 114.6 mm
- net +3.3V: track 0.00 -> 40.2 mm
- net /motorA/MA: track 0.00 -> 39.7 mm
- net GND: track 0.00 -> 36.0 mm
- net +BATT: track 0.00 -> 34.2 mm
- net /mcu/~{RESET}: track 0.00 -> 32.5 mm, vias 0 -> 2
- net Net-(U3-ECHO): track 0.00 -> 24.9 mm
- net /mcu/TIM3_CH1: track 0.00 -> 24.4 mm, vias 0 -> 2
- net /mcu/OUT_B9: track 0.00 -> 23.5 mm
- net /mcu/TIM3_CH2: track 0.00 -> 21.1 mm, vias 0 -> 2
- net /mcu/TIM15_CH1: track 0.00 -> 14.7 mm, vias 0 -> 2
- net /mcu/SWO: track 0.00 -> 14.1 mm
- net /mcu/SWDCLK: track 0.00 -> 13.5 mm
- net Net-(U5-REF): track 0.00 -> 13.2 mm
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- added copper zone on F.Cu, net GND

Commit message: save
Parts:
- Rsnsa1, Rsnsb1: footprint Resistor_SMD:R_0603_1608Metric -> Resistor_SMD:R_2512_6332Metric
- moved C1 26.0 mm to (164.7, 87.0), turned to 0 degrees
- moved C6 21.0 mm to (154.6, 91.8), turned to -90 degrees
- moved C3 16.6 mm to (152.8, 91.9), turned to -90 degrees
- moved Rsnsb1 11.3 mm to (141.3, 111.2)
- moved Rsnsa1 10.4 mm to (154.7, 110.7), turned to -90 degrees
- moved C8 7.85 mm to (155.0, 61.9)
- moved C11 7.19 mm to (151.0, 65.9), turned to 90 degrees
- moved C2 6.81 mm to (147.2, 78.5), turned to 90 degrees
- moved C4 3.73 mm to (143.3, 86.3)
- moved C5 2.83 mm to (143.3, 82.7)
- moved C10 2.54 mm to (133.0, 74.6)
- moved R8 1.79 mm to (153.9, 76.8)
- moved R9 1.79 mm to (149.2, 76.8)
- moved R12 1.79 mm to (150.8, 76.8)
- moved R1 1.79 mm to (152.5, 76.8)
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Connections:
- Rsnsb1 pad 1: Net-(U5-SENSEA) -> +BATT
- U5 pad 4: Net-(U5-SENSEA) -> +BATT
Routing:
- net +BATT: track 34.2 -> 113.7 mm, vias 0 -> 10
- net /mcu/TIM2_CH1: track 126.9 -> 69.5 mm, vias 0 -> 2
- net /mcu/TIM2_CH2: track 114.6 -> 75.1 mm, vias 0 -> 2
- net /motorB/MB: track 0.00 -> 38.3 mm, vias 0 -> 4
- net /motorB/MA: track 0.00 -> 32.4 mm, vias 0 -> 6
- net +3.3V: track 40.2 -> 25.6 mm
- net /motorA/MB: track 0.00 -> 13.5 mm, vias 0 -> 3
- net Net-(U5-SENSEB): track 2.26 -> 11.2 mm, vias 0 -> 2
- net GND: track 36.0 -> 29.8 mm, vias 0 -> 12
- net /mcu/IN_B2: track 12.7 -> 7.63 mm
- net /mcu/~{RESET}: track 32.5 -> 36.8 mm
- net Net-(U5-SENSEA): track 2.28 -> 0.00 mm
- net Net-(U1-PB6): track 3.72 -> 5.90 mm
- net Net-(U5-REF): track 13.2 -> 15.1 mm
- net /mcu/BOOT0: track 3.39 -> 5.05 mm
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- added copper zone on B.Cu, net GND
- removed copper zone on F.Cu, net GND
