File: mm_motor_control.kicad_sch (KiCad schematic)
At the start: 10 parts, among them U5 STSPIN240

Commit message: save
Parts:
- Rsnsa1, Rsnsb1: footprint Resistor_SMD:R_0603_1608Metric -> Resistor_SMD:R_2512_6332Metric
Changed lines of the file:
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@@
       (effects (font (size 1.27 1.27)) (justify left))
     )
-    (property "Footprint" "Resistor_SMD:R_0603_1608Metric" (at 168.402 109.22 90)
+    (property "Footprint" "Resistor_SMD:R_2512_6332Metric" (at 168.402 109.22 90)
       (effects (font (size 1.27 1.27)) hide)
     )
@@
       (effects (font (size 1.27 1.27)) (justify left))
     )
-    (property "Footprint" "Resistor_SMD:R_0603_1608Metric" (at 179.832 107.95 90)
-      (effects (font (size 1.27 1.27)) hide)
-    )
+    (property "Footprint" "Resistor_SMD:R_2512_6332Metric" (at 179.832 107.95 90)
+      (effects (font (size 1.27 1.27)) hide)
+    )
